Commit message: simplified model

File: vehicles/models/selfie/macros.xacro (robot description, xacro)
@@ -2,31 +2,33 @@
 <robot name="selfie" xmlns:xacro="http://www.ros.org/wiki/xacro">
 <!-- inertial parameter macros -->
+<xacro:property name="wheelRadius" value="${0.04}" />
+<xacro:property name="wheelWidth" value="${0.03 }" />
+<xacro:property name="wheelMass" value="${100 }" />
+<xacro:property name="hingeRadius" value="${0.1 }" />
+<xacro:property name="hingeMass" value="${1 }" />
+<xacro:property name="chassisX" value="${0.22 }" />
+<xacro:property name="chassisY" value="${0.2 }" />
+<xacro:property name="chassisZ" value="${0.1 }" />
+<xacro:property name="chassisMass" value="${1000}" />
 <xacro:macro name="chassis_inertial_params">
-  <origin xyz="0.1477 0 0" rpy="0 0 0" />
-  <mass value="10.0" />
-  <inertia ixx="0.010609" ixy="0"          ixz="0"
-                          iyy="0.050409"   iyz="0"
-                                           izz="0.05865" />
+  <origin xyz="${chassisX/2} 0 0" rpy="0 0 0" />
+  <mass value="${chassisMass}" />
+  <inertia ixx="${chassisMass*(chassisY*chassisY + chassisZ*chassisZ)/12}" ixy="0"          ixz="0"
+                          iyy="${chassisMass*(chassisX*chassisX + chassisZ*chassisZ)/12}"   iyz="0"
+                                           izz="${chassisMass*(chassisY*chassisY + chassisX*chassisX)/12}" />
 </xacro:macro>
-<xacro:macro name="left_wheels_inertial_params">
-  <origin xyz="0 0 -0.0225" rpy="0 0 0" />
-  <mass value="0.34055" />
-  <inertia ixx="0.00026046" ixy="0"          ixz="0"
-                            iyy="0.00026046" iyz="0"
-                                             izz="0.00041226" />
-</xacro:macro>
-<xacro:macro name="right_wheels_inertial_params">
-  <origin xyz="0 0 0.0225" rpy="0 0 0" />
-  <mass value="0.34055" />
-  <inertia ixx="0.00026046" ixy="0"          ixz="0"
-                            iyy="0.00026046" iyz="0"
-                                             izz="0.00041226" />
+<xacro:macro name="wheel_inertial_params">
+  <origin xyz="0 0 0" rpy="0 0 0" />
+  <mass value="${wheelMass}" />
+  <inertia ixx="${wheelMass*(3*wheelRadius*wheelRadius+wheelWidth*wheelWidth)/12}" ixy="0"          ixz="0"
+                            iyy="${wheelMass*(3*wheelRadius*wheelRadius+wheelWidth*wheelWidth)/12}" iyz="0"
+                                             izz="${wheelMass*wheelRadius*wheelRadius/2}" />
 </xacro:macro>
 <xacro:macro name="steering_hinge_inertial_params">
   <origin xyz="0 0 0" rpy="0 0 0" />
-  <mass value="0.100" />
-  <inertia ixx="4E-06" ixy="0"           ixz="0"
-                            iyy="4E-06"  iyz="0"
-                                              izz="4E-06" />
+  <mass value="${hingeMass}" />
+  <inertia ixx="${2*hingeMass*hingeRadius*hingeRadius/3}" ixy="0"           ixz="0"
+                            iyy="${2*hingeMass*hingeRadius*hingeRadius/3}"  iyz="0"
+                                              izz="${2*hingeMass*hingeRadius*hingeRadius/3}" />
 </xacro:macro>
 <xacro:macro name="hokuyo_inertial_params">
@@ -39,55 +41,13 @@
 <!-- geometry macros -->
 <xacro:macro name="chassis_geometry">
-  <origin xyz="0.11 0 0" rpy="0 0 0" /> <!-- origin xyz="-0.08 0 0" rpy="0 0 0"-->
+  <origin xyz="${chassisX/2} 0 0" rpy="0 0 0" /> <!-- origin xyz="-0.08 0 0" rpy="0 0 0"-->
   <geometry>
-    <mesh filename="package://gazebo_selfie_sim/vehicles/models/selfie/meshes/my_chasis.STL" />
+    <mesh filename="package://gazebo_selfie_sim/vehicles/models/selfie/meshes/my_chasis.STL"/>
   </geometry>
 </xacro:macro>
-<xacro:macro name="left_rear_wheel_geometry">
-  <origin xyz="0 0 0" rpy="0 0 0" />
+<xacro:macro name="wheel_geometry">
+  <origin xyz="0 0 0.0" rpy="0 0 0" />
   <geometry>
-    <mesh filename="package://gazebo_selfie_sim/vehicles/models/selfie/meshes/selfie_left_rear_wheel.STL" />
-  </geometry>
-</xacro:macro>
-<xacro:macro name="right_rear_wheel_geometry">
-  <origin xyz="0 0 0" rpy="0 0 0" />
-  <geometry>
-    <mesh filename="package://gazebo_selfie_sim/vehicles/models/selfie/meshes/selfie_right_rear_wheel.STL" />
-  </geometry>
-</xacro:macro>
-<xacro:macro name="left_front_wheel_geometry">
-  <origin xyz="0 0 0" rpy="0 0 0" />
-  <geometry>
-    <mesh filename="package://gazebo_selfie_sim/vehicles/models/selfie/meshes/selfie_left_front_wheel.STL" />
-  </geometry>
-</xacro:macro>
-<xacro:macro name="right_front_wheel_geometry">
-  <origin xyz="0 0 0" rpy="0 0 0" />
-  <geometry>
-    <mesh filename="package://gazebo_selfie_sim/vehicles/models/selfie/meshes/selfie_right_front_wheel.STL" />
-  </geometry>
-</xacro:macro>
-<xacro:macro name="left_steering_hinge_geometry">
-  <origin xyz="0 0 0" rpy="0 0 0" />
-  <geometry>
-    <mesh filename="package://gazebo_selfie_sim/vehicles/models/selfie/meshes/left_steering_hinge.STL" />
-  </geometry>
-</xacro:macro>
-<xacro:macro name="right_steering_hinge_geometry">
-  <origin xyz="0 0 0" rpy="0 0 0" />
-  <geometry>
-    <mesh filename="package://gazebo_selfie_sim/vehicles/models/selfie/meshes/right_steering_hinge.STL" />
-  </geometry>
-</xacro:macro>
-<xacro:macro name="left_wheels_collision_geometry">
-  <origin xyz="0 0 -0.0225" rpy="0 0 0" />
-  <geometry>
-    <cylinder length="0.0333" radius="0.03" />
-  </geometry>
-</xacro:macro>
-<xacro:macro name="right_wheels_collision_geometry">
-  <origin xyz="0 0 0.0225" rpy="0 0 0" />
-  <geometry>
-    <cylinder length="0.0333" radius="0.03" />  <!-- changed from 0.045   -->
+    <cylinder radius="${wheelRadius}" length="${wheelWidth}"/>
   </geometry>
 </xacro:macro>

File: vehicles/models/selfie/selfie.xacro (robot description, xacro)
@@ -4,7 +4,10 @@
   <xacro:include filename="$(find gazebo_selfie_sim)/vehicles/models/selfie/selfie.gazebo" />
   <xacro:include filename="$(find gazebo_selfie_sim)/vehicles/models/selfie/materials.xacro" />
-  <!-- Add chassis and it's inertia link -->
-  <link name="base_link" />
-  <link name="chassis">
+  <link name="selfie">
+  </link>
+  <link name="base_link">
+    <inertial>
+      <xacro:chassis_inertial_params />
+    </inertial>
     <visual>
       <xacro:chassis_geometry/>
@@ -12,18 +15,8 @@
     </visual>
   </link>
-  <joint name="base_link_joint" type="fixed">
-    <origin xyz="0 0 0.05" rpy="0 0 0" />
-    <parent link="base_link" />
-    <child link="chassis" />
-  </joint>
-  <link name="chassis_inertia">
-    <inertial>
-      <xacro:chassis_inertial_params />
-    </inertial>
-  </link>
-  <joint name="chassis_inertia_joint" type="fixed">
-    <origin xyz="0 0 0" rpy="0 0 0" />
-    <parent link="chassis" />
-    <child link="chassis_inertia" />
+  <joint name="base_link" type="fixed">
+    <origin xyz="0 0 0" rpy="0 0 0" /> <!-- 0.325-->
+    <parent link="selfie" />
+    <child link="base_link" />
   </joint>
   <!-- Add the left rear steering hinge with its joints and tranmissions -->
@@ -32,15 +25,11 @@
       <xacro:steering_hinge_inertial_params />
     </inertial>
-    <visual>
-      <xacro:left_steering_hinge_geometry />
-      <material name="grey" />
-    </visual>
   </link>
   <joint name="left_rear_steering_hinge_joint" type="revolute">
-    <origin xyz="0 0.06 0" rpy="0 1.5708 0" /> <!-- 0.325-->
-    <parent link="chassis" />
+    <origin xyz="0 ${chassisY/2} 0" rpy="0 0 0" /> <!-- 0.325-->
+    <parent link="base_link" />
     <child link="left_rear_steering_hinge" />
-    <axis xyz="-1 0 0" />
-    <limit lower="-1.0" upper="1.0" effort="10" velocity="1000" />
+    <axis xyz="0 0 1" />
+    <limit lower="-1.0" upper="1.0" effort="10000" velocity="1000" />
   </joint>
   <xacro:steering_hinge_transmission name="left_rear_steering_hinge" />
@@ -50,15 +39,11 @@
       <xacro:steering_hinge_inertial_params />
     </inertial>
-    <visual>
-      <xacro:right_steering_hinge_geometry />
-      <material name="grey" />
-    </visual>
-  </link>
-  <joint name="right_rear_steering_hinge_joint" type="continuous">
-    <origin xyz="0 -0.06 0" rpy="0 1.5708 0" />  <!-- 0.325-->
-    <parent link="chassis" />
+  </link>
+  <joint name="right_rear_steering_hinge_joint" type="revolute">
+    <origin xyz="0 ${-chassisY/2} 0" rpy="0 0 0" />  <!-- 0.325-->
+    <parent link="base_link" />
     <child link="right_rear_steering_hinge" />
-    <axis xyz="-1 0 0" />
-    <limit lower="-1.0" upper="1.0" effort="10" velocity="1000" />
+    <axis xyz="0 0 1" />
+    <limit lower="-1.0" upper="1.0" effort="10000" velocity="1000" />
   </joint>
   <xacro:steering_hinge_transmission name="right_rear_steering_hinge" />
@@ -66,20 +51,20 @@
   <link name="left_rear_wheel">
     <inertial>
-      <xacro:left_wheels_inertial_params />
-    </inertial>
-    <visual>
-      <xacro:left_rear_wheel_geometry />
-      <material name="black" />
-    </visual>
-    <collision>
-      <xacro:left_wheels_collision_geometry />
+      <xacro:wheel_inertial_params />
+    </inertial>
+    <visual>
+      <xacro:wheel_geometry />
+      <material name="black" />
+    </visual>
+    <collision>
+      <xacro:wheel_geometry />
     </collision>
   </link>
   <joint name="left_rear_wheel_joint" type="continuous">
-    <origin xyz="0 0 0" rpy="1.5708 0 0" />
+    <origin xyz="0 0 0" rpy="-1.5708 0 0" />
     <parent link="left_rear_steering_hinge" />
     <child link="left_rear_wheel" />
-    <axis xyz="0 0 -1" />
-    <limit effort="10" velocity="1000" />
+    <axis xyz="0 0 1" />
+    <limit effort="10000" velocity="1000" />
   </joint>
   <xacro:wheel_transmission name="left_rear_wheel" />
@@ -87,20 +72,20 @@
   <link name="right_rear_wheel">
     <inertial>
-      <xacro:right_wheels_inertial_params />
-    </inertial>
-    <visual>
-      <xacro:right_rear_wheel_geometry />
-      <material name="black" />
-    </visual>
-    <collision>
-      <xacro:right_wheels_collision_geometry />
+      <xacro:wheel_inertial_params />
+    </inertial>
+    <visual>
+      <xacro:wheel_geometry />
+      <material name="black" />
+    </visual>
+    <collision>
+      <xacro:wheel_geometry />
     </collision>
   </link>
   <joint name="right_rear_wheel_joint" type="continuous">
-    <origin xyz="0 0 0" rpy="1.5708 0 0" />
+    <origin xyz="0 0 0" rpy="-1.5708 0 0" />
     <parent link="right_rear_steering_hinge" />
     <child link="right_rear_wheel" />
-    <axis xyz="0 0 -1" />
-    <limit effort="10" velocity="1000" />
+    <axis xyz="0 0 1" />
+    <limit effort="10000" velocity="1000" />
   </joint>
   <xacro:wheel_transmission name="right_rear_wheel" />
@@ -110,15 +95,11 @@
       <xacro:steering_hinge_inertial_params />
     </inertial>
-    <visual>
-      <xacro:left_steering_hinge_geometry />
-      <material name="grey" />
-    </visual>
   </link>
   <joint name="left_front_steering_hinge_joint" type="revolute">
-    <origin xyz="0.225 0.06 0" rpy="0 1.5708 0" /> <!-- 0.325-->
-    <parent link="chassis" />
+    <origin xyz="${chassisX} ${chassisY/2} 0" rpy="0 0 0" /> <!-- 0.325-->
+    <parent link="base_link" />
     <child link="left_front_steering_hinge" />
-    <axis xyz="-1 0 0" />
-    <limit lower="-1.0" upper="1.0" effort="10" velocity="1000" />
+    <axis xyz="0 0 1" />
+    <limit lower="-1.0" upper="1.0" effort="10000" velocity="1000" />
   </joint>
   <xacro:steering_hinge_transmission name="left_front_steering_hinge" />
@@ -128,15 +109,11 @@
       <xacro:steering_hinge_inertial_params />
     </inertial>
-    <visual>
-      <xacro:right_steering_hinge_geometry />
-      <material name="grey" />
-    </visual>
-  </link>
-  <joint name="right_front_steering_hinge_joint" type="continuous">
-    <origin xyz="0.225 -0.06 0" rpy="0 1.5708 0" />  <!-- 0.325-->
-    <parent link="chassis" />
+  </link>
+  <joint name="right_front_steering_hinge_joint" type="revolute">
+    <origin xyz="${chassisX} -${chassisY/2} 0" rpy="0 0 0" />  <!-- 0.325-->
+    <parent link="base_link" />
     <child link="right_front_steering_hinge" />
-    <axis xyz="-1 0 0" />
-    <limit lower="-1.0" upper="1.0" effort="10" velocity="1000" />
+    <axis xyz="0 0 1" />
+    <limit lower="-1.0" upper="1.0" effort="10000" velocity="1000" />
   </joint>
   <xacro:steering_hinge_transmission name="right_front_steering_hinge" />
@@ -144,20 +121,20 @@
   <link name="left_front_wheel">
     <inertial>
-      <xacro:left_wheels_inertial_params />
-    </inertial>
-    <visual>
-      <xacro:left_front_wheel_geometry />
-      <material name="black" />
-    </visual>
-    <collision>
-      <xacro:left_wheels_collision_geometry />
+      <xacro:wheel_inertial_params />
+    </inertial>
+    <visual>
+      <xacro:wheel_geometry />
+      <material name="black" />
+    </visual>
+    <collision>
+      <xacro:wheel_geometry />
     </collision>
   </link>
   <joint name="left_front_wheel_joint" type="continuous">
-    <origin xyz="0 0 0" rpy="1.5708 0 0" />
+    <origin xyz="0 0 0" rpy="-1.5708 0 0" />
     <parent link="left_front_steering_hinge" />
     <child link="left_front_wheel" />
-    <axis xyz="0 0 -1" />
-    <limit effort="10" velocity="1000" />
+    <axis xyz="0 0 1" />
+    <limit effort="10000" velocity="1000" />
   </joint>
   <xacro:wheel_transmission name="left_front_wheel" />
@@ -165,20 +142,20 @@
   <link name="right_front_wheel">
     <inertial>
-      <xacro:right_wheels_inertial_params />
-    </inertial>
-    <visual>
-      <xacro:right_front_wheel_geometry />
-      <material name="black" />
-    </visual>
-    <collision>
-      <xacro:right_wheels_collision_geometry />
+      <xacro:wheel_inertial_params />
+    </inertial>
+    <visual>
+      <xacro:wheel_geometry />
+      <material name="black" />
+    </visual>
+    <collision>
+      <xacro:wheel_geometry />
     </collision>
   </link>
   <joint name="right_front_wheel_joint" type="continuous">
-    <origin xyz="0 0 0" rpy="1.5708 0 0" />
+    <origin xyz="0 0 0" rpy="-1.5708 0 0" />
     <parent link="right_front_steering_hinge" />
     <child link="right_front_wheel" />
-    <axis xyz="0 0 -1" />
-    <limit effort="10" velocity="1000"/>
+    <axis xyz="0 0 1" />
+    <limit effort="10000" velocity="1000"/>
   </joint>
   <xacro:wheel_transmission name="right_front_wheel" />
@@ -204,5 +181,5 @@
   <joint name="hokuyo_joint" type="fixed">
     <origin xyz="0.2 0.0 0.075" rpy="0 0 0"/>
-    <parent link="chassis" />
+    <parent link="base_link" />
     <child link="laser" />
     <axis xyz="0 0 1" />
@@ -220,5 +197,5 @@
   <joint name="base_mast_joint" type="fixed">
     <origin xyz="0 0 0" rpy="0 0 0"/>
-    <parent link="chassis"/>
+    <parent link="base_link"/>
     <child link="mast_link"/>
     <axis xyz="0 0 1"/>
@@ -239,4 +216,11 @@
       <material name="black"/>
     </visual>
+  </link>
+  <joint name="imu_base_joint" type="fixed">
+    <origin xyz="0.15 0 0" rpy="0 0 0"/>
+    <parent link="base_link"/>
+    <child link="imu_link"/>
+  </joint>
+  <link name="imu_link">
   </link>
   <joint name="camera_joint" type="fixed">

Commit message: car dimentions params

File: vehicles/models/selfie/macros.xacro (robot description, xacro)
@@ -2,33 +2,24 @@
 <robot name="selfie" xmlns:xacro="http://www.ros.org/wiki/xacro">
 <!-- inertial parameter macros -->
-<xacro:property name="wheelRadius" value="${0.04}" />
-<xacro:property name="wheelWidth" value="${0.03 }" />
-<xacro:property name="wheelMass" value="${100 }" />
-<xacro:property name="hingeRadius" value="${0.1 }" />
-<xacro:property name="hingeMass" value="${1 }" />
-<xacro:property name="chassisX" value="${0.22 }" />
-<xacro:property name="chassisY" value="${0.2 }" />
-<xacro:property name="chassisZ" value="${0.1 }" />
-<xacro:property name="chassisMass" value="${1000}" />
 <xacro:macro name="chassis_inertial_params">
-  <origin xyz="${chassisX/2} 0 0" rpy="0 0 0" />
-  <mass value="${chassisMass}" />
-  <inertia ixx="${chassisMass*(chassisY*chassisY + chassisZ*chassisZ)/12}" ixy="0"          ixz="0"
-                          iyy="${chassisMass*(chassisX*chassisX + chassisZ*chassisZ)/12}"   iyz="0"
-                                           izz="${chassisMass*(chassisY*chassisY + chassisX*chassisX)/12}" />
+  <origin xyz="${chassis_x/2} 0 0" rpy="0 0 0" />
+  <mass value="${chassis_mass}" />
+  <inertia ixx="${chassis_mass*(chassis_y*chassis_y + chassis_z*chassis_z)/12}" ixy="0"          ixz="0"
+                          iyy="${chassis_mass*(chassis_x*chassis_x + chassis_z*chassis_z)/12}"   iyz="0"
+                                           izz="${chassis_mass*(chassis_y*chassis_y + chassis_x*chassis_x)/12}" />
 </xacro:macro>
 <xacro:macro name="wheel_inertial_params">
   <origin xyz="0 0 0" rpy="0 0 0" />
-  <mass value="${wheelMass}" />
-  <inertia ixx="${wheelMass*(3*wheelRadius*wheelRadius+wheelWidth*wheelWidth)/12}" ixy="0"          ixz="0"
-                            iyy="${wheelMass*(3*wheelRadius*wheelRadius+wheelWidth*wheelWidth)/12}" iyz="0"
-                                             izz="${wheelMass*wheelRadius*wheelRadius/2}" />
+  <mass value="${wheel_mass}" />
+  <inertia ixx="${wheel_mass*(3*wheel_radius*wheel_radius+wheel_width*wheel_width)/12}" ixy="0"          ixz="0"
+                            iyy="${wheel_mass*(3*wheel_radius*wheel_radius+wheel_width*wheel_width)/12}" iyz="0"
+                                             izz="${wheel_mass*wheel_radius*wheel_radius/2}" />
 </xacro:macro>
 <xacro:macro name="steering_hinge_inertial_params">
   <origin xyz="0 0 0" rpy="0 0 0" />
-  <mass value="${hingeMass}" />
-  <inertia ixx="${2*hingeMass*hingeRadius*hingeRadius/3}" ixy="0"           ixz="0"
-                            iyy="${2*hingeMass*hingeRadius*hingeRadius/3}"  iyz="0"
-                                              izz="${2*hingeMass*hingeRadius*hingeRadius/3}" />
+  <mass value="${hinge_mass}" />
+  <inertia ixx="${2*hinge_mass*hinge_radius*hinge_radius/3}" ixy="0"           ixz="0"
+                            iyy="${2*hinge_mass*hinge_radius*hinge_radius/3}"  iyz="0"
+                                              izz="${2*hinge_mass*hinge_radius*hinge_radius/3}" />
 </xacro:macro>
 <xacro:macro name="hokuyo_inertial_params">
@@ -41,5 +32,5 @@
 <!-- geometry macros -->
 <xacro:macro name="chassis_geometry">
-  <origin xyz="${chassisX/2} 0 0" rpy="0 0 0" /> <!-- origin xyz="-0.08 0 0" rpy="0 0 0"-->
+  <origin xyz="${chassis_x/2} 0 0" rpy="0 0 0" /> <!-- origin xyz="-0.08 0 0" rpy="0 0 0"-->
   <geometry>
     <mesh filename="package://gazebo_selfie_sim/vehicles/models/selfie/meshes/my_chasis.STL"/>
@@ -49,5 +40,5 @@
   <origin xyz="0 0 0.0" rpy="0 0 0" />
   <geometry>
-    <cylinder radius="${wheelRadius}" length="${wheelWidth}"/>
+    <cylinder radius="${wheel_radius}" length="${wheel_width}"/>
   </geometry>
 </xacro:macro>

File: vehicles/models/selfie/selfie.xacro (robot description, xacro)
@@ -1,7 +1,10 @@
 <?xml version="1.0"?>
 <robot name="selfie" xmlns:xacro="http://www.ros.org/wiki/xacro">
+  <xacro:include filename="$(find gazebo_selfie_sim)/vehicles/models/selfie/load_params.xacro" />
   <xacro:include filename="$(find gazebo_selfie_sim)/vehicles/models/selfie/macros.xacro" />
   <xacro:include filename="$(find gazebo_selfie_sim)/vehicles/models/selfie/selfie.gazebo" />
   <xacro:include filename="$(find gazebo_selfie_sim)/vehicles/models/selfie/materials.xacro" />
+<xacro:property name="yaml_file" value="$(find gazebo_selfie_sim)/vehicles/models/selfie/config/dims.yaml" />
+<xacro:property name="props" value="${load_yaml(yaml_file)}"/>
   <link name="selfie">
   </link>
@@ -27,5 +30,5 @@
   </link>
   <joint name="left_rear_steering_hinge_joint" type="revolute">
-    <origin xyz="0 ${chassisY/2} 0" rpy="0 0 0" /> <!-- 0.325-->
+    <origin xyz="0 ${chassis_y/2} 0" rpy="0 0 0" /> <!-- 0.325-->
     <parent link="base_link" />
     <child link="left_rear_steering_hinge" />
@@ -41,5 +44,5 @@
   </link>
   <joint name="right_rear_steering_hinge_joint" type="revolute">
-    <origin xyz="0 ${-chassisY/2} 0" rpy="0 0 0" />  <!-- 0.325-->
+    <origin xyz="0 ${-chassis_y/2} 0" rpy="0 0 0" />  <!-- 0.325-->
     <parent link="base_link" />
     <child link="right_rear_steering_hinge" />
@@ -97,5 +100,5 @@
   </link>
   <joint name="left_front_steering_hinge_joint" type="revolute">
-    <origin xyz="${chassisX} ${chassisY/2} 0" rpy="0 0 0" /> <!-- 0.325-->
+    <origin xyz="${chassis_x} ${chassis_y/2} 0" rpy="0 0 0" /> <!-- 0.325-->
     <parent link="base_link" />
     <child link="left_front_steering_hinge" />
@@ -111,5 +114,5 @@
   </link>
   <joint name="right_front_steering_hinge_joint" type="revolute">
-    <origin xyz="${chassisX} -${chassisY/2} 0" rpy="0 0 0" />  <!-- 0.325-->
+    <origin xyz="${chassis_x} -${chassis_y/2} 0" rpy="0 0 0" />  <!-- 0.325-->
     <parent link="base_link" />
     <child link="right_front_steering_hinge" />
