Commit message: add new model with distance sensor

File: vehicles/sensors/camera/properties.xacro (robot description, xacro)
@@ -1,4 +1,4 @@
 <?xml version="1.0"?>
-<robot name="selfie">
+<robot name="$(arg robot_name)">
   <xacro:macro name="camera_params"  xmlns:xacro="http://www.ros.org/wiki/xacro">
     <horizontal_fov>1.58</horizontal_fov>     <!--0.8709216071359963-->

File: vehicles/sensors/distance/properties.xacro (robot description, xacro)
@@ -1,19 +1,19 @@
 <?xml version="1.0"?>
 <robot name="$(arg robot_name)">
-  <xacro:macro name="lidar_params" xmlns:xacro="http://www.ros.org/wiki/xacro">
-    <visualize>false</visualize>
-    <update_rate>10</update_rate>
+  <xacro:macro name="distance_params" xmlns:xacro="http://www.ros.org/wiki/xacro">
+    <visualize>true</visualize>
+    <update_rate>100</update_rate>
     <ray>
       <scan>
         <horizontal>
-          <samples>780</samples>
+          <samples>1</samples>
           <resolution>1</resolution>
-          <min_angle>-2.3561944902</min_angle>
-          <max_angle>2.3561944902</max_angle>
+          <min_angle>0.0</min_angle>
+          <max_angle>0.1</max_angle>
         </horizontal>
       </scan>
       <range>
-        <min>0.06</min>
-        <max>6.0</max>
+        <min>0.01</min>
+        <max>5.0</max>
         <resolution>0.005</resolution>
       </range>
