Commit message: add depth camera

File: vehicles/models/selfie2021/selfie2021.xacro (robot description, xacro)
@@ -338,3 +338,21 @@
   <link name="distance_link">
   </link>
+  <joint name="depth_camera_joint" type="fixed">
+    <origin xyz="0.02 0 0.1" rpy="0 -${3.14/2} 0"/>
+    <parent link="mast_link"/>
+    <child link="depth_camera_link"/>
+  </joint>
+  <link name="depth_camera_link">
+    <visual>
+      <geometry>
+        <cylinder radius="0.03"  length="0.025"/>
+      </geometry>
+    </visual>
+  </link>
+  <joint name="depth_camera_lens_joint" type="fixed">
+    <origin xyz="0 0 0.03" rpy="0 ${3.14/2} 0"/>
+    <parent link="depth_camera_link"/>
+    <child link="depth_camera_lens"/>
+  </joint>
+  <link name="depth_camera_lens" />
 </robot>

Commit message: fix frames of depth camera

File: vehicles/models/selfie2021/selfie2021.xacro (robot description, xacro)
@@ -285,5 +285,5 @@
       </geometry>
       <material name="black"/>
-      <origin xyz="0 0 0.1051" rpy="0 0 3.14"/><!--0.26-->
+      <origin xyz="0 0 0.1051" rpy="0 0 0"/><!--0.26-->
     </visual>
   </link>
@@ -344,4 +344,7 @@
   </joint>
   <link name="depth_camera_link">
+    <inertial>
+      <xacro:steering_hinge_inertial_params />
+    </inertial>
     <visual>
       <geometry>
@@ -356,3 +359,9 @@
   </joint>
   <link name="depth_camera_lens" />
+  <joint name="depth_camera_lens_optical_joint" type="fixed">
+    <origin xyz="0 0 0.03" rpy="${-3.14/2} 0 ${-3.14/2}"/>
+    <parent link="depth_camera_lens"/>
+    <child link="depth_camera_lens_optical"/>
+  </joint>
+  <link name="depth_camera_lens_optical" />
 </robot>

Commit message: Feature/updated model

File: vehicles/models/selfie2021/selfie2021.xacro (robot description, xacro)
@@ -243,39 +243,4 @@
     <child link="left_back_indicator" />
   </joint>
-  <!-- Add Hokuyo laser scanner -->
-  <link name="laser_base">
-    <inertial>
-      <xacro:hokuyo_inertial_params />
-    </inertial>
-    <collision>
-      <origin xyz="0 0 0" rpy="0 0 0"/>
-      <geometry>
-        <box size="0.05 0.05 0.05"/>
-      </geometry>
-    </collision>
-    <visual>
-      <origin xyz="0 0 0" rpy="0 0 0"/>
-      <geometry>
-        <mesh filename="package://gazebo_selfie_sim/vehicles/sensors/hokuyo/meshes/hokuyo.dae" scale="0.7 0.7 0.7"/>
-        <material name="grey" />
-      </geometry>
-    </visual>
-  </link>
-  <joint name="hokuyo_joint" type="fixed">
-    <origin xyz="0.24 0.0 0.04" rpy="0 0 0"/>
-    <parent link="base_link" />
-    <child link="laser_base" />
-    <axis xyz="0 0 1" />
-  </joint>
-  <link name="laser">
-    <inertial>
-      <xacro:hokuyo_inertial_params />
-    </inertial>
-  </link>
-  <joint name="laser_joint" type="fixed">
-    <origin xyz="0.0 0.0 0.015" rpy="0 0 0"/>
-    <parent link="laser_base" />
-    <child link="laser" />
-  </joint>
   <!-- camera -->
   <link name="mast_link">
@@ -285,5 +250,5 @@
       </geometry>
       <material name="black"/>
-      <origin xyz="0 0 0.1051" rpy="0 0 3.14"/><!--0.26-->
+      <origin xyz="0 0 0.1051" rpy="0 0 0"/><!--0.26-->
     </visual>
   </link>
@@ -331,3 +296,37 @@
   <link name="lens_link">
   </link>
+  <joint name="distance_joint" type="fixed">
+    <origin xyz="0 ${-wheel_y - 0.01} 0" rpy="0 0 -${3.14/2}"/>
+    <parent link="base_link"/>
+    <child link="distance_link"/>
+  </joint>
+  <link name="distance_link">
+  </link>
+  <joint name="depth_camera_joint" type="fixed">
+    <origin xyz="0.02 0 0.1" rpy="0 -${3.14/2} 0"/>
+    <parent link="mast_link"/>
+    <child link="depth_camera_link"/>
+  </joint>
+  <link name="depth_camera_link">
+    <inertial>
+      <xacro:steering_hinge_inertial_params />
+    </inertial>
+    <visual>
+      <geometry>
+        <cylinder radius="0.03"  length="0.025"/>
+      </geometry>
+    </visual>
+  </link>
+  <joint name="depth_camera_lens_joint" type="fixed">
+    <origin xyz="0 0 0.03" rpy="0 ${3.14/2} 0"/>
+    <parent link="depth_camera_link"/>
+    <child link="depth_camera_lens"/>
+  </joint>
+  <link name="depth_camera_lens" />
+  <joint name="depth_camera_lens_optical_joint" type="fixed">
+    <origin xyz="0 0 0.03" rpy="${-3.14/2} 0 ${-3.14/2}"/>
+    <parent link="depth_camera_lens"/>
+    <child link="depth_camera_lens_optical"/>
+  </joint>
+  <link name="depth_camera_lens_optical" />
 </robot>

File: vehicles/sensors/distance/properties.xacro (robot description, xacro)
@@ -1,19 +1,19 @@
 <?xml version="1.0"?>
 <robot name="$(arg robot_name)">
-  <xacro:macro name="lidar_params" xmlns:xacro="http://www.ros.org/wiki/xacro">
+  <xacro:macro name="distance_params" xmlns:xacro="http://www.ros.org/wiki/xacro">
     <visualize>false</visualize>
-    <update_rate>10</update_rate>
+    <update_rate>100</update_rate>
     <ray>
       <scan>
         <horizontal>
-          <samples>780</samples>
+          <samples>1</samples>
           <resolution>1</resolution>
-          <min_angle>-2.3561944902</min_angle>
-          <max_angle>2.3561944902</max_angle>
+          <min_angle>0.0</min_angle>
+          <max_angle>0.1</max_angle>
         </horizontal>
       </scan>
       <range>
-        <min>0.06</min>
-        <max>6.0</max>
+        <min>0.01</min>
+        <max>5.0</max>
         <resolution>0.005</resolution>
       </range>
